File: kicad_source/RP2040LoRaTracker/RP2040LoRaTracker.kicad_pcb (KiCad board)
At the start: 2 copper layers, 28 x 87 mm, 69 parts, among them J1 USB_B_Micro, J2 BM04B-SRSS-TB, Q1 NTR4171P, SW1 SW_Push, SW2 SW_Push, SW3 SW_SPDT, U1 RP2040, U2 Ai-Thinker-Ra-01, U3 NEO-M8N, U4 W25Q16JVSS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

Commit message: updated some values in schematic, added comments, updated schematic pdf
Parts:
- R11, R7: value 0R -> DNI
Changed lines of the file:
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@@
 	(title_block
 		(title "RP2040LoRaTracker")
-		(date "2025-04-01")
+		(date "2025-04-20")
 		(rev "0.1")
 		(company "generationmake")
@@
 			(net 79 "unconnected-(U3-V_BCKP-Pad22)")
 			(pinfunction "V_BCKP")
-			(pintype "power_in")
+			(pintype "power_in+no_connect")
 		)
 		(pad "23" smd roundrect
@@
 			)
 		)
-		(property "Value" "0R"
+		(property "Value" "DNI"
 			(at 0 1.43 90)
 			(layer "F.Fab")
@@
 		(tags "capacitor")
 		(property "Reference" "C22"
-			(at 0 1.5 360)
+			(at 0 1.5 0)
 			(layer "F.SilkS")
 			(effects
@@
 		)
 		(property "Value" "2.2 uF"
-			(at 0 1.43 360)
+			(at 0 1.43 0)
 			(layer "F.Fab")
 			(effects
@@
 		)
 		(fp_text user "${REFERENCE}"
-			(at 0 0 360)
+			(at 0 0 0)
 			(layer "F.Fab")
 			(effects
@@
 			)
 		)
-		(property "Value" "0R"
+		(property "Value" "DNI"
 			(at 0 1.43 0)
 			(layer "F.Fab")
@@
 			(net 48 "unconnected-(U1-GPIO3-Pad5)")
 			(pinfunction "GPIO3")
-			(pintype "bidirectional")
+			(pintype "bidirectional+no_connect")
 		)
 		(pad "6" smd roundrect
@@
 			(net 38 "unconnected-(U1-GPIO6-Pad8)")
 			(pinfunction "GPIO6")
-			(pintype "bidirectional")
+			(pintype "bidirectional+no_connect")
 		)
 		(pad "9" smd roundrect
@@
 			(net 53 "unconnected-(U1-GPIO7-Pad9)")
 			(pinfunction "GPIO7")
-			(pintype "bidirectional")
+			(pintype "bidirectional+no_connect")
 		)
 		(pad "10" smd roundrect
@@
 			(net 60 "unconnected-(U1-GPIO8-Pad11)")
 			(pinfunction "GPIO8")
-			(pintype "bidirectional")
+			(pintype "bidirectional+no_connect")
 		)
 		(pad "12" smd roundrect
@@
 			(net 35 "unconnected-(U1-GPIO11-Pad14)")
 			(pinfunction "GPIO11")
-			(pintype "bidirectional")
+			(pintype "bidirectional+no_connect")
 		)
 		(pad "15" smd roundrect
@@
 			(net 41 "unconnected-(U1-GPIO12-Pad15)")
 			(pinfunction "GPIO12")
-			(pintype "bidirectional")
+			(pintype "bidirectional+no_connect")
 		)
 		(pad "16" smd roundrect
@@
 			(net 59 "unconnected-(U1-GPIO13-Pad16)")
 			(pinfunction "GPIO13")
-			(pintype "bidirectional")
+			(pintype "bidirectional+no_connect")
 		)
 		(pad "17" smd roundrect
@@
 			(net 62 "unconnected-(U1-GPIO14-Pad17)")
 			(pinfunction "GPIO14")
-			(pintype "bidirectional")
+			(pintype "bidirectional+no_connect")
 		)
 		(pad "18" smd roundrect
@@
 			(net 32 "unconnected-(U1-GPIO15-Pad18)")
 			(pinfunction "GPIO15")
-			(pintype "bidirectional")
+			(pintype "bidirectional+no_connect")
 		)
 		(pad "19" smd roundrect
@@
 			(net 37 "unconnected-(U1-SWCLK-Pad24)")
 			(pinfunction "SWCLK")
-			(pintype "input")
+			(pintype "input+no_connect")
 		)
 		(pad "25" smd roundrect
@@
 			(net 39 "unconnected-(U1-SWD-Pad25)")
 			(pinfunction "SWD")
-			(pintype "bidirectional")
+			(pintype "bidirectional+no_connect")
 		)
 		(pad "26" smd roundrect
@@
 			(net 50 "unconnected-(U1-GPIO17-Pad28)")
 			(pinfunction "GPIO17")
-			(pintype "bidirectional")
+			(pintype "bidirectional+no_connect")
 		)
 		(pad "29" smd roundrect
@@
 			(net 30 "unconnected-(U1-GPIO20-Pad31)")
 			(pinfunction "GPIO20")
-			(pintype "bidirectional")
+			(pintype "bidirectional+no_connect")
 		)
 		(pad "32" smd roundrect
@@
 			(net 47 "unconnected-(U1-GPIO21-Pad32)")
 			(pinfunction "GPIO21")
-			(pintype "bidirectional")
+			(pintype "bidirectional+no_connect")
 		)
 		(pad "33" smd roundrect
@@
 			(net 29 "unconnected-(U1-GPIO22-Pad34)")
 			(pinfunction "GPIO22")
-			(pintype "bidirectional")
+			(pintype "bidirectional+no_connect")
 		)
 		(pad "35" smd roundrect
@@
 			(net 27 "unconnected-(U1-GPIO23-Pad35)")
 			(pinfunction "GPIO23")
-			(pintype "bidirectional")
+			(pintype "bidirectional+no_connect")
 		)
 		(pad "36" smd roundrect
@@
 			(net 45 "unconnected-(U1-GPIO24-Pad36)")
 			(pinfunction "GPIO24")
-			(pintype "bidirectional")
+			(pintype "bidirectional+no_connect")
 		)
 		(pad "37" smd roundrect
@@
 			(net 28 "unconnected-(U1-GPIO26_ADC0-Pad38)")
 			(pinfunction "GPIO26_ADC0")
-			(pintype "bidirectional")
+			(pintype "bidirectional+no_connect")
 		)
 		(pad "39" smd roundrect
@@
 			(net 46 "unconnected-(U1-GPIO27_ADC1-Pad39)")
 			(pinfunction "GPIO27_ADC1")
-			(pintype "bidirectional")
+			(pintype "bidirectional+no_connect")
 		)
 		(pad "40" smd roundrect
@@
 			(net 33 "unconnected-(U1-GPIO28_ADC2-Pad40)")
 			(pinfunction "GPIO28_ADC2")
-			(pintype "bidirectional")
+			(pintype "bidirectional+no_connect")
 		)
 		(pad "41" smd roundrect
@@
 			(net 49 "unconnected-(U1-GPIO29_ADC3-Pad41)")
 			(pinfunction "GPIO29_ADC3")
-			(pintype "bidirectional")
+			(pintype "bidirectional+no_connect")
 		)
 		(pad "42" smd roundrect
