File: kicad_source/RP2040LoRaTracker/RP2040LoRaTracker.kicad_pcb (KiCad board)
At the start: 2 copper layers, 28 x 87 mm, 73 parts, among them J1 USB_B_Micro, J2 BM04B-SRSS-TB, Q1 NTR4171P, SW1 SW_Push, SW2 SW_Push, SW3 SW_SPDT, U1 RP2040, U2 Ai-Thinker-Ra-01, U3 NEO-M8N, U4 W25Q16JVSS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

Commit message: added compatibility for LoRa module Ra-01S, added R20 and R21
Parts:
- added R20: DNI, Resistor_SMD:R_0603_1608Metric, F.Cu at (128.0, 90.5)
- added R21: DNI, Resistor_SMD:R_0603_1608Metric, F.Cu at (128.0, 93.7)
- moved C10 1.20 mm to (132.7, 118.8)
- moved C8 1.20 mm to (132.7, 117.3)
Connections:
- U1 pad 31: unconnected-(U1-GPIO20-Pad31) -> /RP2040/LORA_DIO1_R
- U1 pad 32: unconnected-(U1-GPIO21-Pad32) -> /RP2040/LORA_BUSY_R
- U2 pad 10: unconnected-(U2-DIO4-Pad10) -> LORA_BUSY
- U2 pad 6: unconnected-(U2-DIO1-Pad6) -> LORA_DIO1
Routing:
- net /RP2040/LORA_DIO1_R: track 0.00 -> 30.9 mm
- net /RP2040/LORA_BUSY_R: track 0.00 -> 28.2 mm
- net LORA_DIO1: track 0.00 -> 26.1 mm, vias 0 -> 2
- net LORA_BUSY: track 0.00 -> 12.9 mm
- net +3V3: track 171.1 -> 176.3 mm
- net GND: track 527.5 -> 525.4 mm
